File: ECE477_Team1/RobotBoard.brd (EAGLE design)
At the start: 101.3 x 81.3 mm, 81 parts, among them IC1L A3967SLB, IC1R A3967SLB

Commit message: Added Antenna
Parts:
- added ANT: 2450AT18A100, Johanson_antenna:2450AT18A100
- moved R1 2.54 mm to (20.3, 31.8)
- moved R2 2.54 mm to (20.3, 34.3)
- moved SW1 2.54 mm to (20.3, 33.0)
Connections:
- new net N$18: ANT.P$1, WIFI.24
Routing:
- net N$18: track 0.00 -> 10.0 mm
- net 3.3V: track 668.8 -> 661.4 mm
- net GND: track 694.8 -> 693.0 mm
Changed lines of the file:
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@@
 <element name="C9" library="SparkFun-2-11-09" package="0603" value=".1uF" x="10.16" y="60.96" rot="MR90"/>
 <element name="C10" library="SparkFun-2-11-09" package="0603" value=".1uF" x="19.05" y="67.31" rot="MR180"/>
-<element name="SW1" library="SparkFun-Electromechanical" package="DIPSWITCH-02" value="" x="20.32" y="35.56" rot="R90"/>
-<element name="R1" library="SparkFun03_30_09" package="C0402" value="1K" x="20.32" y="34.29" rot="MR180"/>
-<element name="R2" library="SparkFun03_30_09" package="C0402" value="1K" x="20.32" y="36.83" rot="MR180"/>
+<element name="SW1" library="SparkFun-Electromechanical" package="DIPSWITCH-02" value="" x="20.32" y="33.02" rot="R90"/>
+<element name="R1" library="SparkFun03_30_09" package="C0402" value="1K" x="20.32" y="31.75" rot="MR180"/>
+<element name="R2" library="SparkFun03_30_09" package="C0402" value="1K" x="20.32" y="34.29" rot="MR180"/>
 <element name="3.3V_REG" library="SparkFun-PowerIC" package="SOT223" value="" x="91.44" y="66.04" rot="R270">
 <attribute name="PROD_ID" value="VREG-08170" x="91.44" y="66.04" size="1.778" layer="27" rot="R270" display="off"/>
@@
 <element name="R4" library="SparkFun03_30_09" package="C0402" value="10K" x="57.785" y="45.72"/>
 <element name="R5" library="SparkFun03_30_09" package="C0402" value="1K" x="28.321" y="60.96" rot="R270"/>
+<element name="ANT" library="Johanson_antenna" package="2450AT18A100" value="2450AT18A100" x="7.62" y="38.1" rot="R180"/>
 </elements>
 <signals>
@@
 <wire x1="38.1" y1="29.21" x2="39.37" y2="30.48" width="0.6096" layer="1"/>
 <contactref element="PROG" pad="3"/>
-<wire x1="24.13" y1="36.83" x2="24.13" y2="34.29" width="0.6096" layer="16"/>
-<wire x1="24.13" y1="34.29" x2="24.13" y2="33.02" width="0.6096" layer="1"/>
-<wire x1="24.13" y1="33.02" x2="25.4" y2="31.75" width="0.6096" layer="1"/>
-<wire x1="25.4" y1="31.75" x2="35.56" y2="31.75" width="0.6096" layer="1"/>
+<wire x1="24.13" y1="31.75" x2="35.56" y2="31.75" width="0.6096" layer="1"/>
 <wire x1="35.56" y1="31.75" x2="36.83" y2="33.02" width="0.6096" layer="1"/>
 <wire x1="27.94" y1="41.91" x2="29.464" y2="41.91" width="0.4064" layer="16"/>
@@
 <wire x1="64.77" y1="43.18" x2="67.31" y2="43.18" width="0.254" layer="16"/>
 <wire x1="67.31" y1="43.18" x2="68.58" y2="44.45" width="0.254" layer="16"/>
+<wire x1="24.13" y1="31.75" x2="24.13" y2="34.29" width="0.6096" layer="1"/>
 </signal>
 <signal name="N$1">
@@
 <contactref element="SW1" pad="3"/>
 <contactref element="R2" pad="1"/>
-<wire x1="19.67" y1="36.83" x2="16.51" y2="36.83" width="0.6096" layer="16"/>
-<via x="16.51" y="36.83" extent="1-16" drill="0.5"/>
-<wire x1="16.51" y1="36.83" x2="16.51" y2="38.1" width="0.4064" layer="1"/>
+<via x="16.51" y="34.29" extent="1-16" drill="0.5"/>
 <wire x1="29.21" y1="40.64" x2="33.02" y2="44.45" width="0.4064" layer="1"/>
-<wire x1="16.51" y1="38.1" x2="17.78" y2="39.37" width="0.4064" layer="1"/>
-<wire x1="17.78" y1="39.37" x2="25.4" y2="39.37" width="0.4064" layer="1"/>
-<wire x1="25.4" y1="39.37" x2="26.67" y2="40.64" width="0.4064" layer="1"/>
 <wire x1="26.67" y1="40.64" x2="29.21" y2="40.64" width="0.4064" layer="1"/>
+<wire x1="19.67" y1="34.29" x2="16.51" y2="34.29" width="0.6096" layer="16"/>
+<wire x1="26.67" y1="40.64" x2="22.86" y2="36.83" width="0.4064" layer="1"/>
+<wire x1="22.86" y1="36.83" x2="19.05" y2="36.83" width="0.4064" layer="1"/>
+<wire x1="19.05" y1="36.83" x2="16.51" y2="34.29" width="0.4064" layer="1"/>
 </signal>
 <signal name="RB4">
@@
 <contactref element="SW1" pad="4"/>
 <contactref element="R1" pad="1"/>
-<wire x1="19.67" y1="34.29" x2="16.51" y2="34.29" width="0.6096" layer="16"/>
-<wire x1="16.51" y1="34.29" x2="15.24" y2="34.29" width="0.4064" layer="1"/>
-<wire x1="15.24" y1="34.29" x2="13.97" y2="35.56" width="0.4064" layer="1"/>
-<wire x1="13.97" y1="35.56" x2="13.97" y2="39.37" width="0.4064" layer="1"/>
-<wire x1="13.97" y1="39.37" x2="15.24" y2="40.64" width="0.4064" layer="1"/>
-<wire x1="15.24" y1="40.64" x2="24.13" y2="40.64" width="0.4064" layer="1"/>
-<wire x1="24.13" y1="40.64" x2="26.67" y2="43.18" width="0.4064" layer="1"/>
 <wire x1="26.67" y1="43.18" x2="29.21" y2="43.18" width="0.4064" layer="1"/>
 <wire x1="29.21" y1="43.18" x2="31.75" y2="45.72" width="0.4064" layer="1"/>
@@
 <wire x1="34.544" y1="46.228" x2="35.306" y2="46.99" width="0.254" layer="1"/>
 <wire x1="35.306" y1="46.99" x2="35.56" y2="46.99" width="0.254" layer="1"/>
+<wire x1="19.67" y1="31.75" x2="16.51" y2="31.75" width="0.6096" layer="16"/>
+<wire x1="26.67" y1="43.18" x2="21.59" y2="38.1" width="0.4064" layer="1"/>
+<wire x1="21.59" y1="38.1" x2="19.05" y2="38.1" width="0.4064" layer="1"/>
+<wire x1="19.05" y1="38.1" x2="16.51" y2="35.56" width="0.4064" layer="1"/>
+<wire x1="16.51" y1="35.56" x2="15.24" y2="35.56" width="0.4064" layer="1"/>
+<wire x1="15.24" y1="35.56" x2="13.97" y2="34.29" width="0.4064" layer="1"/>
+<wire x1="13.97" y1="34.29" x2="13.97" y2="33.02" width="0.4064" layer="1"/>
+<wire x1="13.97" y1="33.02" x2="15.24" y2="31.75" width="0.4064" layer="1"/>
+<wire x1="15.24" y1="31.75" x2="16.51" y2="31.75" width="0.4064" layer="1"/>
 </signal>
 <signal name="RB5">
@@
 <contactref element="R2" pad="2"/>
 <contactref element="R1" pad="2"/>
-<wire x1="20.97" y1="36.83" x2="21.587" y2="36.87303125" width="0.6096" layer="16"/>
-<wire x1="21.59" y1="36.87603125" x2="21.59" y2="48.26" width="0.6096" layer="16"/>
 <wire x1="21.59" y1="48.26" x2="20.74" y2="49.11" width="0.6096" layer="16"/>
 <wire x1="20.74" y1="49.11" x2="20.32" y2="49.11" width="0.6096" layer="16"/>
@@
 <wire x1="34.91" y1="4.43" x2="33.02" y2="4.43" width="0.6096" layer="1"/>
 <contactref element="PROG" pad="2"/>
-<wire x1="21.59" y1="36.87603125" x2="21.587" y2="36.87303125" width="0.6096" layer="16"/>
-<wire x1="20.97" y1="36.83" x2="20.97" y2="34.29" width="0.6096" layer="16"/>
 <wire x1="27.686" y1="44.45" x2="28.956" y2="44.45" width="0.4064" layer="16"/>
 <wire x1="28.956" y1="44.45" x2="29.718" y2="45.212" width="0.4064" layer="16"/>
@@
 <wire x1="54.05" y1="47.55" x2="53.34" y2="48.26" width="0.254" layer="1"/>
 <wire x1="54.61" y1="48.26" x2="54.61" y2="48.68" width="0.254" layer="16"/>
+<wire x1="20.97" y1="31.75" x2="20.97" y2="34.29" width="0.6096" layer="16"/>
+<wire x1="22.86" y1="27.94" x2="22.86" y2="29.21" width="0.6096" layer="16"/>
+<wire x1="22.86" y1="29.21" x2="20.97" y2="31.1" width="0.6096" layer="16"/>
+<wire x1="20.97" y1="31.1" x2="20.97" y2="31.75" width="0.6096" layer="16"/>
 </signal>
 <signal name="N$4">
@@
 <wire x1="28.321" y1="64.731" x2="28.36" y2="64.77" width="0.4064" layer="1"/>
 </signal>
+<signal name="N$18">
+<contactref element="WIFI" pad="24"/>
+<contactref element="ANT" pad="P$1"/>
+<wire x1="15.24" y1="42.926" x2="15.24" y2="39.37" width="0.8128" layer="1"/>
+<wire x1="15.24" y1="39.37" x2="13.97" y2="38.1" width="0.8128" layer="1"/>
+<wire x1="13.97" y1="38.1" x2="9.32" y2="38.1" width="0.8128" layer="1"/>
+</signal>
 </signals>
