File: ECE477_Team1/RobotBoard.sch (EAGLE design)
At the start: 81 parts, among them IC1L A3967SLB, IC1R A3967SLB

Commit message: Added Antenna
Parts:
- added ANT: 2450AT18A100, Johanson_antenna:2450AT18A100
Connections:
- new net N$18: ANT.P$1, WIFI.ANT
Changed lines of the file:
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@@
 <part name="GND4" library="SparkFun-Aesthetics" deviceset="GND" device=""/>
 <part name="R5" library="SparkFun03_30_09" deviceset="RESISTOR" device="0402" value="1K"/>
+<part name="ANT" library="Johanson_antenna" deviceset="2450AT18A100" device=""/>
 </parts>
 <sheets>
@@
 <instance part="GND4" gate="1" x="73.66" y="10.16"/>
 <instance part="R5" gate="G$1" x="-91.44" y="48.26" rot="R180"/>
+<instance part="ANT" gate="G$1" x="154.94" y="58.42"/>
 </instances>
 <busses>
@@
 </segment>
 </net>
+<net name="N$18" class="0">
+<segment>
+<pinref part="WIFI" gate="G$1" pin="ANT"/>
+<wire x1="162.56" y1="27.94" x2="154.94" y2="27.94" width="0.1524" layer="91"/>
+<wire x1="154.94" y1="27.94" x2="154.94" y2="53.34" width="0.1524" layer="91"/>
+<pinref part="ANT" gate="G$1" pin="P$1"/>
+</segment>
+</net>
