File: ECE477_Team1/RobotBoard_v2.1.brd (EAGLE design)
At the start: 101.6 x 81.3 mm, 86 parts, among them IC1L A3967SLB, IC1R A3967SLB, IC5 5

Commit message: Added Battery
Parts:
- added BAT1: (no value), SparkFun-Electromechanical:BATTCOM_20MM_PTH
- added D1, D3: CGRM4001-G, diode:SOD-123_MINI-SMA
- renumbered PWR12 to PWR
Connections:
- new net N$4: BAT1.1, D3.A
- new net SKSDJIOJ: 3.3V_REG.2, 3.3V_REG.4, C2.1, D1.A
- net 3.3V: now also D1.C, D3.C; no longer 3.3V_REG.2, 3.3V_REG.4, C2.1
- net GND: now also BAT1.2
Routing:
- net SKSDJIOJ: track 0.00 -> 13.9 mm
- net 3.3V: track 646.9 -> 655.0 mm, vias 19 -> 20
- net N$4: track 0.00 -> 2.43 mm
- net N$18: track 10.0 -> 9.26 mm
Other:
- board text added: "ECE477 Team 1--Nathan Tornquist--Mark Harlan--TJ Root--Josh Hannan"
- board text removed: "Team 1--Nathan Tornquist--Mark Harlan--TJ Root--Josh Hannan"
