File: ECE477_Team1/RobotBoard_v2.1.sch (EAGLE design)
At the start: 86 parts, among them IC1L A3967SLB, IC1R A3967SLB, IC5 5

Commit message: Added Battery
Parts:
- added BAT1: (no value), SparkFun-Electromechanical:BATTERY20PTH
- added D1, D3: CGRM4001-G, diode:CGRM4001-G
- renumbered PWR12 to PWR
Connections:
- new net N$4: BAT1.+, D3.A
- new net SKSDJIOJ: 3.3V_REG.OUT, 3.3V_REG.OUT@1, C2.1, D1.A
- net 3.3V: now also D1.C, D3.C; no longer 3.3V_REG.OUT, 3.3V_REG.OUT@1, C2.1
- net GND: now also BAT1.-
Changed lines of the file:
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@@
 <?xml version="1.0" encoding="utf-8"?>
 <!DOCTYPE eagle SYSTEM "eagle.dtd">
-<eagle version="6.1">
+<eagle version="7.2.0">
 <drawing>
 <settings>
@@
 <part name="CAM" library="SparkFun-Connectors" deviceset="M05" device="LOCK"/>
 <part name="WIFI" library="SparkFun-RF" deviceset="RN171" device="RN171"/>
-<part name="PWR12" library="SparkFun-Connectors" deviceset="M02" device="PTH"/>
+<part name="PWR" library="SparkFun-Connectors" deviceset="M02" device="PTH"/>
 <part name="U$2" library="SparkFun-Connectors" deviceset="M08X2" device=""/>
 <part name="U$3" library="SparkFun-Connectors" deviceset="M08X2" device=""/>
@@
 <part name="CO2" library="SparkFun-2-11-09" deviceset="CAP" device="0603" value="20pF"/>
 <part name="GND5" library="SparkFun-Aesthetics" deviceset="GND" device=""/>
+<part name="D1" library="diode" deviceset="CGRM400*-G" device="" technology="1"/>
+<part name="D3" library="diode" deviceset="CGRM400*-G" device="" technology="1"/>
+<part name="BAT1" library="SparkFun-Electromechanical" deviceset="BATTERY" device="20PTH"/>
 </parts>
 <sheets>
@@
 <instance part="CAM" gate="G$1" x="111.76" y="0"/>
 <instance part="WIFI" gate="G$1" x="182.88" y="22.86"/>
-<instance part="PWR12" gate="G$1" x="93.98" y="137.16" rot="R180"/>
+<instance part="PWR" gate="G$1" x="93.98" y="137.16" rot="R180"/>
 <instance part="U$2" gate="G$1" x="-35.56" y="48.26"/>
 <instance part="U$3" gate="G$1" x="27.94" y="-12.7" rot="R90"/>
@@
 <instance part="CO2" gate="G$1" x="53.34" y="-20.32"/>
 <instance part="GND5" gate="1" x="48.26" y="-25.4"/>
+<instance part="D1" gate="G$1" x="139.7" y="101.6"/>
+<instance part="D3" gate="G$1" x="154.94" y="96.52" rot="R90"/>
+<instance part="BAT1" gate="G$1" x="154.94" y="86.36" rot="R270"/>
 </instances>
 <busses>
@@
 <segment>
 <pinref part="GND32" gate="1" pin="GND"/>
-<pinref part="PWR12" gate="G$1" pin="2"/>
+<pinref part="PWR" gate="G$1" pin="2"/>
 <wire x1="83.82" y1="134.62" x2="86.36" y2="134.62" width="0.1524" layer="91"/>
 <pinref part="C5" gate="G$1" pin="-"/>
@@
 <wire x1="132.08" y1="91.44" x2="132.08" y2="81.28" width="0.1524" layer="91"/>
 <wire x1="132.08" y1="81.28" x2="114.3" y2="81.28" width="0.1524" layer="91"/>
+<pinref part="BAT1" gate="G$1" pin="-"/>
+<wire x1="154.94" y1="81.28" x2="132.08" y2="81.28" width="0.1524" layer="91"/>
 </segment>
 <segment>
@@
 </segment>
 <segment>
-<pinref part="3.3V_REG" gate="G$1" pin="OUT"/>
-<pinref part="3.3V_REG" gate="G$1" pin="OUT@1"/>
-<wire x1="121.92" y1="101.6" x2="121.92" y2="99.06" width="0.1524" layer="91"/>
-<wire x1="121.92" y1="101.6" x2="132.08" y2="101.6" width="0.1524" layer="91"/>
-<junction x="121.92" y="101.6"/>
-<pinref part="C2" gate="G$1" pin="1"/>
-<wire x1="132.08" y1="101.6" x2="132.08" y2="99.06" width="0.1524" layer="91"/>
+<pinref part="D3" gate="G$1" pin="C"/>
+<pinref part="D1" gate="G$1" pin="C"/>
+<wire x1="154.94" y1="99.06" x2="154.94" y2="101.6" width="0.1524" layer="91"/>
+<wire x1="154.94" y1="101.6" x2="142.24" y2="101.6" width="0.1524" layer="91"/>
 </segment>
 </net>
 <net name="N$19" class="0">
 <segment>
-<pinref part="PWR12" gate="G$1" pin="1"/>
+<pinref part="PWR" gate="G$1" pin="1"/>
 <wire x1="86.36" y1="137.16" x2="81.28" y2="137.16" width="0.1524" layer="91"/>
 <wire x1="81.28" y1="137.16" x2="81.28" y2="121.92" width="0.1524" layer="91"/>
@@
 </segment>
 </net>
+<net name="N$4" class="0">
+<segment>
+<pinref part="BAT1" gate="G$1" pin="+"/>
+<pinref part="D3" gate="G$1" pin="A"/>
+<wire x1="154.94" y1="91.44" x2="154.94" y2="93.98" width="0.1524" layer="91"/>
+</segment>
+</net>
+<net name="SKSDJIOJ" class="0">
+<segment>
+<pinref part="3.3V_REG" gate="G$1" pin="OUT"/>
+<pinref part="3.3V_REG" gate="G$1" pin="OUT@1"/>
+<wire x1="121.92" y1="101.6" x2="121.92" y2="99.06" width="0.1524" layer="91"/>
+<wire x1="121.92" y1="101.6" x2="132.08" y2="101.6" width="0.1524" layer="91"/>
+<junction x="121.92" y="101.6"/>
+<pinref part="C2" gate="G$1" pin="1"/>
+<wire x1="132.08" y1="101.6" x2="132.08" y2="99.06" width="0.1524" layer="91"/>
+<pinref part="D1" gate="G$1" pin="A"/>
+<wire x1="137.16" y1="101.6" x2="132.08" y2="101.6" width="0.1524" layer="91"/>
+</segment>
+</net>
